File: Diy-Macropad.kicad_pcb (KiCad board)
At the start: 2 copper layers, 70 x 100 mm, 28 parts, among them J1 Conn_01x04, SW1 RotaryEncoder_Switch, U1 MCU_Seeed_XIAO_RP2040

Commit message: added copper ground
Parts:
- added G***: LOGO, Orbit logo:Orbit_logo, F.Cu at (127.0, 57.0)
- H1, H2, H3, H4: footprint MountingHole:MountingHole_2.2mm_M2 -> MountingHole:MountingHole_2.2mm_M2_DIN965_Pad
Connections:
- SW1 pad C: Rotary C -> GND
- U1 pad 13: Rotary C -> GND
Routing:
- added copper zone on B.Cu, net GND
Other:
- board text added: "Made with Love By Sumit Patil"
